File: Hardware/CoffeePal.sch (EAGLE design)
At the start: 27 parts, among them U1 ATTINY85SOIC-8, U2 BH1745NUC-E2WSON008X2120, U3 TP143305-1PIETZO, U4 CMPT3904ETRPBFREESOT23

Commit message: Drew traces and created boom
Parts:
- added U$3: UTBULT_DESIGN1, lib:UTBULT_DESIGN1
- D1: value DIODE1 -> 1N4448W-7-F; LINK (none) -> https://www.mouser.se/ProductDetail/Diodes-Incorporated/1N4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; MPN (none) -> 1N4448W-7-F; SUPPLIER (none) -> Mouser
- renumbered U$1 to U5
Connections:
- net SCL/SCK renamed I2C_P
- net SDA/MOSI renamed I2C_N
